File: KiCad/interfaces.sch (KiCad schematic (older format))
At the start: 27 parts, among them J10 5-2337992-8, J2 DF17(4.0)-50DS-0.5V(57), J3 L834-1G1T-S7, J8 1-2199230-6, T8 WE-RJ45_7499511611A

Commit message: Remove rejected ethernet ports
Parts:
- removed J3: L834-1G1T-S7, antmicro-footprints:BEL_L834-1G1T-S7, symbol antmicroModularConnectorsJacksWithMagnetics:L834-1G1T-S7
- removed T8: WE-RJ45_7499511611A, antmicro-footprints:7499511611A, symbol antmicroModularConnectorsJacksWithMagnetics:WE-RJ45_7499511611A
Changed lines of the file:
@@
 L antmicroModularConnectorsJacksWithMagnetics:5-2337992-8 J10
 U 1 1 628CFF58
-P 13150 2275
-F 0 "J10" H 15150 2696 60  0000 C CNN
-F 1 "5-2337992-8" H 15150 2590 60  0000 C CNN
-F 2 "antmicro-footprints:5-2337992-8" H 15150 225 60  0001 C CNN
-F 3 "" H 14600 2125 60  0000 C CNN
-F 4 "5-2337992-8" H 15150 2492 50  0000 C CNN "MPN"
-F 5 "TE Connectivity" H 15150 2401 50  0000 C CNN "Manufacturer"
-	1    13150 2275
+P 13325 4975
+F 0 "J10" H 15325 5396 60  0000 C CNN
+F 1 "5-2337992-8" H 15325 5290 60  0000 C CNN
+F 2 "antmicro-footprints:5-2337992-8" H 15325 2925 60  0001 C CNN
+F 3 "" H 14775 4825 60  0000 C CNN
+F 4 "5-2337992-8" H 15325 5192 50  0000 C CNN "MPN"
+F 5 "TE Connectivity" H 15325 5101 50  0000 C CNN "Manufacturer"
+	1    13325 4975
 	1    0    0    -1
 $EndComp
-$Comp
-L antmicroModularConnectorsJacksWithMagnetics:WE-RJ45_7499511611A T8
-U 1 1 62931A77
-P 17900 3200
-F 0 "T8" H 17950 4317 50  0000 C CNN
-F 1 "WE-RJ45_7499511611A" H 17950 4226 50  0000 C CNN
-F 2 "antmicro-footprints:7499511611A" H 17900 3200 50  0001 L BNN
-F 3 "" H 17900 3200 50  0001 L BNN
-F 4 "7499511611A" H 17900 3200 50  0001 L BNN "VALUE"
-F 5 "green/orange-yellow" H 17900 3200 50  0001 L BNN "LED"
-F 6 "1" H 17900 3200 50  0001 L BNN "PORTS"
-F 7 "PoE+ (up to 600 mA)" H 17900 3200 50  0001 L BNN "POE"
-F 8 "https://www.we-online.com/catalog/datasheet/7499511611A.pdf" H 17900 3200 50  0001 L BNN "DATASHEET-URL"
-F 9 "7499511611A" H 17900 3200 50  0001 L BNN "MPN"
-F 10 "WURTH ELEKTRONIK" H 17900 3200 50  0001 L BNN "Manufacturer"
-	1    17900 3200
-	1    0    0    -1
-$EndComp
-$Comp
-L antmicroModularConnectorsJacksWithMagnetics:L834-1G1T-S7 J3
-U 1 1 62934D46
-P 20200 2900
-F 0 "J3" H 20530 2946 50  0000 L CNN
-F 1 "L834-1G1T-S7" H 20530 2855 50  0000 L CNN
-F 2 "antmicro-footprints:BEL_L834-1G1T-S7" H 20200 2900 50  0001 L BNN
-F 3 "" H 20200 2900 50  0001 L BNN
-F 4 "L834-1G1T-S7" H 20200 2900 50  0001 L BNN "MPN"
-F 5 "Bel Magnetic Solutions" H 20200 2900 50  0001 L BNN "Manufacturer"
-	1    20200 2900
-	1    0    0    -1
-$EndComp
